Commit message: Changed the robot design
+Removed front wheels from the design to adapt to differential drive plugin. 
+Added caster wheels to the design
+Fixed robot base collision and visual size Z mismatch

Resolves: skid steer design for differential drive plugin.

File: project2/my_robot/urdf/my_robot.xacro (robot description, xacro)
@@ -4,10 +4,4 @@
 	<gazebo reference='robot_base'>
 		<material> Gazebo/Grey </material>
-	</gazebo>
-	<gazebo reference='LeftFrontWheel'>
-		<material> Gazebo/FlatBlack </material>
-	</gazebo>
-	<gazebo reference='RightFrontWheel'>
-		<material> Gazebo/FlatBlack </material>
 	</gazebo>
 	<gazebo reference='LeftBackWheel'>
@@ -29,7 +23,19 @@
    	</visual>
 	<visual name = 'robot_LidarPlate'>
-        	<origin xyz = '0 0 0.15' rpy = '0 0 0' />
+        	<origin xyz = '0 0 0.1' rpy = '0 0 0' />
         	<geometry> <box size='0.2 0.2 0.35'/> </geometry>
    	</visual>
+	<visual name='front_caster_visual'>
+      	<origin xyz="0.7 0 -0.2" rpy=" 0 0 0"/>
+      	<geometry>
+        	<sphere radius="0.06"/>
+     	 </geometry>
+        </visual>
+	<collision name='front_caster_collision'>
+      	<origin xyz="0.7 0 -0.2" rpy=" 0 0 0"/>
+      		<geometry>
+        		<sphere radius="0.06"/>
+      		</geometry>
+    	</collision>
     	<collision name = 'collision' >
         	<origin xyz = '0 0 0' rpy = '0 0 0' />
@@ -41,34 +47,4 @@
         	<inertia ixx="0.1" ixy="0" ixz="0" iyy="0.1" iyz="0" izz="0.1"/>
     	</inertial>
-    </link>
-    <link name="LeftFrontWheel">
-    	<visual name='LeftFrontWheel_visual'>
-        	<origin xyz = '0 0 0' rpy = '0 1.5707 1.5707' />
-        	<geometry> <cylinder radius='0.3' length='0.07'/> </geometry>
-    	</visual>
-        <collision name = 'collision'>
-        	<origin xyz = '0 0 0' rpy = '1.5707 1.5707 0' />
-        	<geometry> <cylinder radius='0.3' length='0.07'/> </geometry>
-        </collision>
-        <inertial>
-        	<origin xyz = '0 0 0' rpy='0 0 0' />
-        	<mass value='5' />
-        	<inertia ixx="0.1" ixy="0" ixz="0" iyy="0.1" iyz="0" izz="0.1" />
-        </inertial>
-    </link>
-    <link name="RightFrontWheel">
-    	<visual name='RightFrontWheel_visual'>
-        	<origin xyz = '0 0 0' rpy = '1.5707 1.5707 0' />
-        	<geometry> <cylinder radius='0.3' length='0.07'/> </geometry>
-    	</visual>
-        <collision name = 'collision'>
-        	<origin xyz = '0 0 0' rpy = '1.5707 1.5707 0' />
-        	<geometry> <cylinder radius='0.3' length='0.07'/> </geometry>
-        </collision>
-        <inertial>
-        	<origin xyz = '0 0 0' rpy='0 0 0' />
-        	<mass value='5' />
-        	<inertia ixx="0.1" ixy="0" ixz="0" iyy="0.1" iyz="0" izz="0.1" />
-        </inertial>
     </link>
     <link name="LeftBackWheel">
@@ -132,20 +108,4 @@
         </inertial>
     </link>
-   <joint type="continuous" name="joint_LeftFrontWheel">
-    <origin xyz="0.8 0.35 0" rpy="0 0 0"/>
-    <child link="LeftFrontWheel"/>
-    <parent link="robot_base"/>
-    <axis xyz="0 1 0" rpy="0 0 0"/>
-    <limit effort="10000" velocity="1000"/>
-    <dynamics damping="1.0" friction="1.0"/>
-  </joint>
-   <joint type="continuous" name="joint_RightFrontWheel">
-    <origin xyz="0.8 -0.35 0" rpy="0 0 0"/>
-    <child link="RightFrontWheel"/>
-    <parent link="robot_base"/>
-    <axis xyz="0 1 0" rpy="0 0 0"/>
-    <limit effort="10000" velocity="1000"/>
-    <dynamics damping="1.0" friction="1.0"/>
-  </joint>
   <joint type="continuous" name="joint_LeftBackWheel">
     <origin xyz="-0.8 0.35 0" rpy="0 0 0"/>

Commit message: Changed Robot dimensions
Changed the robot dimensions to make it proportional.

Resolves: Robot design requirements; robot doesn't have smooth motion while turning due to bad proportion.

File: project2/my_robot/urdf/my_robot.xacro (robot description, xacro)
@@ -20,12 +20,12 @@
 	<visual name = 'robot_base_visual'>
         	<origin xyz = '0 0 0' rpy = '0 0 0' />
-        	<geometry> <box size='2 0.6 0.3'/> </geometry>
+        	<geometry> <box size='0.8 0.4 0.2'/> </geometry>
    	</visual>
 	<visual name = 'robot_LidarPlate'>
         	<origin xyz = '0 0 0.1' rpy = '0 0 0' />
-        	<geometry> <box size='0.2 0.2 0.35'/> </geometry>
+        	<geometry> <box size='0.2 0.2 0.15'/> </geometry>
    	</visual>
 	<visual name='front_caster_visual'>
-      	<origin xyz="0.7 0 -0.2" rpy=" 0 0 0"/>
+      	<origin xyz="0.3 0 -0.2" rpy=" 0 0 0"/>
       	<geometry>
         	<sphere radius="0.06"/>
@@ -40,5 +40,5 @@
     	<collision name = 'collision' >
         	<origin xyz = '0 0 0' rpy = '0 0 0' />
-        	<geometry> <box size='2 0.6 0.3'/> </geometry>
+        	<geometry> <box size='0.8 0.4 0.2'/> </geometry>
     	</collision>
     	<inertial>
@@ -51,9 +51,9 @@
     	<visual name='LeftBackWheel_visual'>
         	<origin xyz = '0 0 0' rpy = '1.5707 1.5707 0' />
-        	<geometry> <cylinder radius='0.3' length='0.07'/> </geometry>
+        	<geometry> <cylinder radius='0.2' length='0.07'/> </geometry>
     	</visual>
         <collision name = 'collision'>
         	<origin xyz = '0 0 0' rpy = '1.5707 1.5707 0' />
-        	<geometry> <cylinder radius='0.3' length='0.07'/> </geometry>
+        	<geometry> <cylinder radius='0.2' length='0.07'/> </geometry>
         </collision>
         <inertial>
@@ -66,9 +66,9 @@
     	<visual name='RightBackWheel_visual'>
         	<origin xyz = '0 0 0' rpy = '1.5707 1.5707 0' />
-        	<geometry> <cylinder radius='0.3' length='0.07'/> </geometry>
+        	<geometry> <cylinder radius='0.2' length='0.07'/> </geometry>
     	</visual>
         <collision name = 'collision'>
         	<origin xyz = '0 0 0' rpy = '1.5707 1.5707 0' />
-        	<geometry> <cylinder radius='0.3' length='0.07'/> </geometry>
+        	<geometry> <cylinder radius='0.2' length='0.07'/> </geometry>
         </collision>
         <inertial>
@@ -109,5 +109,5 @@
     </link>
   <joint type="continuous" name="joint_LeftBackWheel">
-    <origin xyz="-0.8 0.35 0" rpy="0 0 0"/>
+    <origin xyz="-0.35 0.35 0" rpy="0 0 0"/>
     <child link="LeftBackWheel"/>
     <parent link="robot_base"/>
@@ -117,5 +117,5 @@
   </joint>
   <joint type="continuous" name="joint_RightBackWheel">
-    <origin xyz="-0.8 -0.35 0" rpy="0 0 0"/>
+    <origin xyz="-0.35 -0.35 0" rpy="0 0 0"/>
     <child link="RightBackWheel"/>
     <parent link="robot_base"/>
@@ -125,5 +125,5 @@
   </joint>
     <joint name ='camera_joint' type = 'fixed'>
-	<origin xyz='0.8 0 0.19' rpy='0 0 0' />
+	<origin xyz='0.35 0 0.12' rpy='0 0 0' />
 	<parent link='robot_base'/>
 	<child link='camera' />

Commit message: Fixed Conflicts

File: project2/my_robot/urdf/my_robot.xacro (robot description, xacro)
@@ -20,12 +20,12 @@
 	<visual name = 'robot_base_visual'>
         	<origin xyz = '0 0 0' rpy = '0 0 0' />
-        	<geometry> <box size='2 0.6 0.3'/> </geometry>
+        	<geometry> <box size='0.8 0.4 0.2'/> </geometry>
    	</visual>
 	<visual name = 'robot_LidarPlate'>
         	<origin xyz = '0 0 0.1' rpy = '0 0 0' />
-        	<geometry> <box size='0.2 0.2 0.35'/> </geometry>
+        	<geometry> <box size='0.2 0.2 0.15'/> </geometry>
    	</visual>
 	<visual name='front_caster_visual'>
-      	<origin xyz="0.7 0 -0.2" rpy=" 0 0 0"/>
+      	<origin xyz="0.3 0 -0.15" rpy=" 0 0 0"/>
       	<geometry>
         	<sphere radius="0.06"/>
@@ -33,5 +33,5 @@
         </visual>
 	<collision name='front_caster_collision'>
-      	<origin xyz="0.7 0 -0.2" rpy=" 0 0 0"/>
+      	<origin xyz="0.3 0 -0.15" rpy=" 0 0 0"/>
       		<geometry>
         		<sphere radius="0.06"/>
@@ -40,5 +40,5 @@
     	<collision name = 'collision' >
         	<origin xyz = '0 0 0' rpy = '0 0 0' />
-        	<geometry> <box size='2 0.6 0.3'/> </geometry>
+        	<geometry> <box size='0.8 0.4 0.2'/> </geometry>
     	</collision>
     	<inertial>
@@ -51,9 +51,9 @@
     	<visual name='LeftBackWheel_visual'>
         	<origin xyz = '0 0 0' rpy = '1.5707 1.5707 0' />
-        	<geometry> <cylinder radius='0.3' length='0.07'/> </geometry>
+        	<geometry> <cylinder radius='0.2' length='0.07'/> </geometry>
     	</visual>
         <collision name = 'collision'>
         	<origin xyz = '0 0 0' rpy = '1.5707 1.5707 0' />
-        	<geometry> <cylinder radius='0.3' length='0.07'/> </geometry>
+        	<geometry> <cylinder radius='0.2' length='0.07'/> </geometry>
         </collision>
         <inertial>
@@ -66,9 +66,9 @@
     	<visual name='RightBackWheel_visual'>
         	<origin xyz = '0 0 0' rpy = '1.5707 1.5707 0' />
-        	<geometry> <cylinder radius='0.3' length='0.07'/> </geometry>
+        	<geometry> <cylinder radius='0.2' length='0.07'/> </geometry>
     	</visual>
         <collision name = 'collision'>
         	<origin xyz = '0 0 0' rpy = '1.5707 1.5707 0' />
-        	<geometry> <cylinder radius='0.3' length='0.07'/> </geometry>
+        	<geometry> <cylinder radius='0.2' length='0.07'/> </geometry>
         </collision>
         <inertial>
@@ -109,5 +109,5 @@
     </link>
   <joint type="continuous" name="joint_LeftBackWheel">
-    <origin xyz="-0.8 0.35 0" rpy="0 0 0"/>
+    <origin xyz="-0.35 0.25 0" rpy="0 0 0"/>
     <child link="LeftBackWheel"/>
     <parent link="robot_base"/>
@@ -117,5 +117,5 @@
   </joint>
   <joint type="continuous" name="joint_RightBackWheel">
-    <origin xyz="-0.8 -0.35 0" rpy="0 0 0"/>
+    <origin xyz="-0.35 -0.25 0" rpy="0 0 0"/>
     <child link="RightBackWheel"/>
     <parent link="robot_base"/>
@@ -125,5 +125,5 @@
   </joint>
     <joint name ='camera_joint' type = 'fixed'>
-	<origin xyz='0.8 0 0.19' rpy='0 0 0' />
+	<origin xyz='0.35 0 0.12' rpy='0 0 0' />
 	<parent link='robot_base'/>
 	<child link='camera' />
@@ -131,5 +131,5 @@
     </joint>
     <joint name ='hokuyo_joint' type = 'fixed'>
-	<origin xyz='0 0 0.35' rpy='0 0 0' />
+	<origin xyz='0 0 0.2' rpy='0 0 0' />
 	<parent link='robot_base'/>
 	<child link='hokuyo' />

Commit message: Update my_robot.xacro

File: project2/my_robot/urdf/my_robot.xacro (robot description, xacro)
@@ -27,5 +27,5 @@
    	</visual>
 	<visual name='front_caster_visual'>
-      	<origin xyz="0.3 0 -0.2" rpy=" 0 0 0"/>
+      	<origin xyz="0.3 0 -0.15" rpy=" 0 0 0"/>
       	<geometry>
         	<sphere radius="0.06"/>
@@ -33,5 +33,5 @@
         </visual>
 	<collision name='front_caster_collision'>
-      	<origin xyz="0.7 0 -0.2" rpy=" 0 0 0"/>
+      	<origin xyz="0.3 0 -0.15" rpy=" 0 0 0"/>
       		<geometry>
         		<sphere radius="0.06"/>
@@ -109,5 +109,5 @@
     </link>
   <joint type="continuous" name="joint_LeftBackWheel">
-    <origin xyz="-0.35 0.35 0" rpy="0 0 0"/>
+    <origin xyz="-0.35 0.25 0" rpy="0 0 0"/>
     <child link="LeftBackWheel"/>
     <parent link="robot_base"/>
@@ -117,5 +117,5 @@
   </joint>
   <joint type="continuous" name="joint_RightBackWheel">
-    <origin xyz="-0.35 -0.35 0" rpy="0 0 0"/>
+    <origin xyz="-0.35 -0.25 0" rpy="0 0 0"/>
     <child link="RightBackWheel"/>
     <parent link="robot_base"/>
@@ -131,5 +131,5 @@
     </joint>
     <joint name ='hokuyo_joint' type = 'fixed'>
-	<origin xyz='0 0 0.35' rpy='0 0 0' />
+	<origin xyz='0 0 0.2' rpy='0 0 0' />
 	<parent link='robot_base'/>
 	<child link='hokuyo' />
